Commit message: added first pass at links

File: template.urdf (robot description, URDF)
Before this commit: robot {body_name:s}, 1 links, 0 joints
Links:
- removed link {body_name:s}
- added link handle, mass {handle_mass}; collision mesh filename={handle_file:s} scale=1 1 1; visual mesh filename={handle_file:s} scale=1. 1. 1.
- added link head, mass {head_mass}; collision mesh filename={head_file:s} scale=1 1 1; visual mesh filename={head_file:s} scale=1. 1. 1.
Joints:
- added joint hammer_joint: type fixed, parent handle, child head
